File: base-station/base-station.kicad_sch (KiCad schematic)
At the start: 37 parts, among them J1 Conn_01x06, J2 USB_C_Receptacle_USB2.0_16P, J3 Conn_01x08, J4 Conn_01x02, J5 Conn_01x02, SW1 SW_Push, SW2 SW_SPST, SW3 SW_SPDT, SW4 SW_Push, SW5 SW_Push, SW6 SW_Push, U1 MCP73832-2-OT, U2 AP2112K-3.3, U3 W25Q128JVS, U4 STM32G431KBTx, Y1 16MHz

Commit message: add layout
Parts:
- removed SW2: SW_SPST, symbol Switch:SW_SPST
- added FID1, FID2, FID3: Fiducial, Fiducial:Fiducial_1mm_Mask3mm, symbol Mechanical:Fiducial
- added H1, H2: MountingHole, MountingHole:MountingHole_3.5mm, symbol Mechanical:MountingHole
- added H3, H4, H5, H6: MountingHole, MountingHole:MountingHole_4mm, symbol Mechanical:MountingHole
- added H7, H8: MountingHole, MountingHole:MountingHole_2.1mm, symbol Mechanical:MountingHole
- added SW2: SW_SPDT, Button_Switch_SMD:SW_SPDT_PCM12, symbol Switch:SW_SPDT
- C1, C10, C13, C2, C3, C4, C5, C6, C7, C8, C9: footprint (none) -> Capacitor_SMD:C_0402_1005Metric
- D1: footprint (none) -> LED_SMD:LED_0805_2012Metric
- FB1, FB2: footprint (none) -> Inductor_SMD:L_0805_2012Metric
- J1: footprint (none) -> Connector_PinHeader_2.54mm:PinHeader_1x06_P2.54mm_Vertical_SMD_Pin1Left
- J2: footprint (none) -> Connector_USB:USB_C_Receptacle_HRO_TYPE-C-31-M-12
- J3: footprint (none) -> Connector_PinHeader_2.54mm:PinHeader_1x08_P2.54mm_Vertical
- J4: footprint (none) -> Connector_JST:JST_PH_S2B-PH-K_1x02_P2.00mm_Horizontal
- J5: footprint (none) -> Connector_PinHeader_2.54mm:PinHeader_1x02_P2.54mm_Vertical
- R1, R2: footprint (none) -> Resistor_SMD:R_0603_1608Metric
- R3, R4, R5: footprint (none) -> Resistor_SMD:R_0805_2012Metric
- SW1: footprint (none) -> Button_Switch_SMD:SW_Push_1P1T_NO_CK_KMR2
- SW3: footprint (none) -> Button_Switch_SMD:SW_SPDT_PCM12
- SW4, SW5, SW6: footprint (none) -> footprints:Kailh_socket_PG1350_optional
- U3: footprint Package_SO:SOIC-8_5.3x5.3mm_P1.27mm -> Package_SO:SOIC-8_3.9x4.9mm_P1.27mm
Connections:
- net VBAT: now also SW2.1 (A)
- net SW_RESET: now reaches C13.1, SW1.1
- net RESET: now reaches SW1.2, U4.4 (PG10)
- net STAT: now reaches R3.1, U1.1 (STAT)
- net PROG: now reaches R4.1, U1.5 (PROG)
- net VIN: now reaches C3.1, U2.1 (VIN), U2.3 (EN)
- net VIN: now also SW2.2 (B)
- net SW_BOOT: now reaches R5.1, SW3.2 (B)
- net SHIELD: now reaches FB1.2, J2.S1 (SHIELD)
- net LED: now reaches D1.1 (K), R3.2
- net CC2: now reaches J2.B5 (CC2), R2.1
- net BOOT: now reaches R5.2, U4.31 (PB8)
- net CC1: now reaches J2.A5 (CC1), R1.1
- no-connect marks 6 -> 7
Other:
- note added: "Board Mounting Holes"
- note added: "Fiducials"
- note added: "LCD Mounting Holes"
- note added: "Magnet Holes"
- note added: "These holes are used to glue small magnets for the magnetic POGO connectors."
- moved on the sheet: D1, R3, R4, R5

Commit message: add mfg files
Parts:
- C1, C2: LCSC PN (none) -> C77004
- C10: LCSC PN (none) -> C541371
- C13, C5, C6: LCSC PN (none) -> C71687
- C3, C4, C8, C9: LCSC PN (none) -> C14445
- C7: LCSC PN (none) -> C77000
- D1: LCSC PN (none) -> C284871
- FB1, FB2: LCSC PN (none) -> C1017
- J2: LCSC PN (none) -> C165948
- J3: LCSC PN (none) -> C190820
- J4: now not fitted; now left out of the parts list
- J5: LCSC PN (none) -> C234182
- R1, R2: LCSC PN (none) -> C23186
- R3: LCSC PN (none) -> C17710
- R4: LCSC PN (none) -> C17604
- R5: LCSC PN (none) -> C17414
- SW1: LCSC PN (none) -> C221675
- SW2, SW3: LCSC PN (none) -> C431540
- SW4, SW5, SW6: now not fitted
- U1: LCSC PN (none) -> C38066
- U2: LCSC PN (none) -> C23380830
- U3: footprint Package_SO:SOIC-8_3.9x4.9mm_P1.27mm -> Package_SO:SOIC-8_5.3x5.3mm_P1.27mm; LCSC PN (none) -> C97521
- U4: LCSC PN (none) -> C529357
